Commit message: velodyne frame

File: social_sim_ros/urdf/jackal/jackal.urdf.xacro (robot description, xacro)
@@ -209,4 +209,10 @@
     <origin xyz="0 0 0.214" />
   </joint>
+  <link name="velodyne"></link>
+  <joint name="velodyne_joint" type="fixed">
+    <parent link="chassis_link" />
+    <child link="velodyne" />
+    <origin xyz="0 0 0.228" />
+  </joint>
   <link name="mid_mount"></link>
   <joint name="mid_mount_joint" type="fixed">
