Commit message: [warthog] rename wheel joints to match driver, make {right,left}_diff_unit_joint fixed for now

File: social_sim_ros/urdf/warthog/warthog.urdf.xacro (robot description, xacro)
@@ -58,5 +58,5 @@
       </collision>
     </link>
-    <joint name="${prefix}_${side}_wheel_joint" type="continuous">
+    <joint name="${prefix}_${side}_wheel" type="continuous">
       <parent link="${side}_diff_unit_link"/>
       <child link="${prefix}_${side}_wheel_link"/>
@@ -75,5 +75,5 @@
     <transmission name="${prefix}_${side}_wheel_trans">
       <type>transmission_interface/SimpleTransmission</type>
-      <joint name="${prefix}_${side}_wheel_joint">
+      <joint name="${prefix}_${side}_wheel">
         <hardwareInterface>hardware_interface/VelocityJointInterface</hardwareInterface>
       </joint>
@@ -115,5 +115,5 @@
       </collision>
     </link>
-    <joint name="${prefix}_${side}_wheel_joint" type="continuous">
+    <joint name="${prefix}_${side}_wheel" type="continuous">
       <parent link="${side}_diff_unit_link"/>
       <child link="${prefix}_${side}_wheel_link"/>
@@ -123,5 +123,5 @@
     <transmission name="${prefix}_${side}_wheel_trans">
       <type>transmission_interface/SimpleTransmission</type>
-      <joint name="${prefix}_${side}_wheel_joint">
+      <joint name="${prefix}_${side}_wheel">
         <hardwareInterface>hardware_interface/VelocityJointInterface</hardwareInterface>
       </joint>
@@ -132,4 +132,5 @@
     </transmission>
   </xacro:macro>
+  <xacro:unless value="$(optenv WARTHOG_TRACKS 0)">
     <xacro:wheel prefix="front" side="left">
       <origin xyz="${axle_x_offset*1} ${axle_y_offset*1} ${axle_z_offset}" rpy="0 0 0" />
@@ -144,4 +145,5 @@
       <origin xyz="${axle_x_offset*-1} ${axle_y_offset*-1} ${axle_z_offset}" rpy="0 0 0" />
     </xacro:wheel>
+  </xacro:unless>
   <xacro:if value="$(optenv WARTHOG_TRACKS 0)">
     <xacro:track prefix="front" side="left">
@@ -201,11 +203,8 @@
       </collision>
     </link>
-    <joint name="${prefix}_diff_unit_joint" type="revolute">
-      <limit upper="0.4" lower="-0.4" effort="100" velocity="1"/>
+    <joint name="${prefix}_diff_unit_joint" type="fixed">
       <parent link="chassis_link"/>
       <child link="${prefix}_diff_unit_link"/>
       <origin xyz="${diff_unit_offset_x} ${diff_unit_offset_y*side} ${diff_unit_offset_z}" rpy="0 0 0" />
-      <axis xyz="0 1 0"/>
-      <dynamics damping="100" friction="0.5"/>
     </joint>
     <gazebo reference="${prefix}_diff_unit_link">
@@ -214,6 +213,6 @@
     </gazebo>
   </xacro:macro>
-  <xacro:diff_unit prefix="left" side="1" left="true"></xacro:diff_unit>
-  <xacro:diff_unit prefix="right" side="-1" left="false"></xacro:diff_unit>
+  <xacro:diff_unit prefix="left" side="1" left="true"/>
+  <xacro:diff_unit prefix="right" side="-1" left="false"/>
   <link name="base_link"></link>
   <joint name="base_link_joint" type="fixed">

Commit message: warthog urdf updated a bit

File: social_sim_ros/urdf/warthog/warthog.urdf.xacro (robot description, xacro)
@@ -59,5 +59,6 @@
     </link>
     <joint name="${prefix}_${side}_wheel" type="continuous">
-      <parent link="${side}_diff_unit_link"/>
+      <!-- <parent link="${side}_diff_unit_link"/> --> <!-- we put tires under chassis_link-->
+      <parent link="chassis_link"/>
       <child link="${prefix}_${side}_wheel_link"/>
       <xacro:insert_block name="joint_pose" />
@@ -101,5 +102,6 @@
     </link>
     <joint name="${prefix}_${side}_track_joint" type="fixed">
-      <parent link="${side}_diff_unit_link"/>
+      <!-- <parent link="${side}_diff_unit_link"/> -->
+      <parent link="chassis_link" />
       <child link="${prefix}_${side}_track_link"/>
       <xacro:insert_block name="joint_pose" />
@@ -116,5 +118,6 @@
     </link>
     <joint name="${prefix}_${side}_wheel" type="continuous">
-      <parent link="${side}_diff_unit_link"/>
+      <!-- <parent link="${side}_diff_unit_link"/> -->
+      <parent link="chassis_link" />
       <child link="${prefix}_${side}_wheel_link"/>
       <xacro:insert_block name="joint_pose" />

Commit message: bring back default urdf, update wheel joint names to match driver

File: social_sim_ros/urdf/warthog/warthog.urdf.xacro (robot description, xacro)
@@ -59,6 +59,5 @@
     </link>
     <joint name="${prefix}_${side}_wheel" type="continuous">
-      <!-- <parent link="${side}_diff_unit_link"/> --> <!-- we put tires under chassis_link-->
-      <parent link="chassis_link"/>
+      <parent link="${side}_diff_unit_link"/>
       <child link="${prefix}_${side}_wheel_link"/>
       <xacro:insert_block name="joint_pose" />
@@ -102,6 +101,5 @@
     </link>
     <joint name="${prefix}_${side}_track_joint" type="fixed">
-      <!-- <parent link="${side}_diff_unit_link"/> -->
-      <parent link="chassis_link" />
+      <parent link="${side}_diff_unit_link"/>
       <child link="${prefix}_${side}_track_link"/>
       <xacro:insert_block name="joint_pose" />
@@ -118,6 +116,5 @@
     </link>
     <joint name="${prefix}_${side}_wheel" type="continuous">
-      <!-- <parent link="${side}_diff_unit_link"/> -->
-      <parent link="chassis_link" />
+      <parent link="${side}_diff_unit_link"/>
       <child link="${prefix}_${side}_wheel_link"/>
       <xacro:insert_block name="joint_pose" />
@@ -207,7 +204,10 @@
     </link>
     <joint name="${prefix}_diff_unit_joint" type="fixed">
+      <limit upper="0.4" lower="-0.4" effort="100" velocity="1"/>
       <parent link="chassis_link"/>
       <child link="${prefix}_diff_unit_link"/>
       <origin xyz="${diff_unit_offset_x} ${diff_unit_offset_y*side} ${diff_unit_offset_z}" rpy="0 0 0" />
+      <axis xyz="0 1 0"/>
+      <dynamics damping="100" friction="0.5"/>
     </joint>
     <gazebo reference="${prefix}_diff_unit_link">
@@ -293,10 +293,4 @@
     <child link="imu_link" />
   </joint>
-  <link name="laser"></link>
-  <joint name="laser_joint" type="fixed">
-    <parent link="chassis_link" />
-    <child link="laser" />
-    <origin xyz="0 0 0.214" />
-  </joint>
   <!-- Bring in simulation data for Gazebo. -->
   <xacro:include filename="$(find warthog_description)/urdf/warthog.gazebo" />

Commit message: add the velodyne frame, update a name

File: social_sim_ros/urdf/warthog/warthog.urdf.xacro (robot description, xacro)
@@ -252,4 +252,10 @@
     </collision>
   </link>
+  <link name="velodyne"></link>
+  <joint name="velodyne_joint" type="fixed">
+    <parent link="top_chassis_link" />
+    <child link="velodyne" />
+    <origin xyz="0 0 0.75" />
+  </joint>
   <link name="top_chassis_link"></link>
   <joint name="top_link_joint" type="fixed">
